Commit message: Prepare for Gazebo visualization
* launch_sim.launch.py: new launch file to launch gazebo and spawn robot
  with a single command
* robot.urdf.xacro: add call to properties.xacro and gazebo_control.xacro
* robot_core.xacro:
  - move properties definition (robot dimensions etc) to a separate file
  - add gazebo tags to define colors for each link
  - add very low friction coefficients mu1 mu2 for caster wheels
* properties.xacro: new file with properties definition
* gazebo_control.xacro: new file with configuration of diff_drive plugin
  for gazebo

File: manolobot_uno/description/robot.urdf.xacro (robot description, xacro)
@@ -1,5 +1,9 @@
 <?xml version="1.0"?>
 <robot xmlns:xacro="http://www.ros.org/wiki/xacro"  name="manolobot_uno">
-    <!-- Core robot description file -->
+    <!-- PROPERTIES -->
+    <xacro:include filename="properties.xacro" />
+    <!-- CORE ROBOT DESCRIPTION -->
     <xacro:include filename="robot_core.xacro" />
+    <!-- GAZEBO -->
+    <xacro:include filename="gazebo_control.xacro" />
 </robot>

File: manolobot_uno/description/robot_core.xacro (robot description, xacro)
@@ -6,26 +6,4 @@
     <!-- INERTIAL MACROS -->
     <xacro:include filename="inertial_macros.xacro" />
-    <!-- PROPERTIES -->
-    <xacro:property name="L_x" value="0.29"/> <!-- box length -->
-    <xacro:property name="L_y" value="0.19"/> <!-- box width -->
-    <xacro:property name="L_z" value="0.124"/> <!-- box height -->
-    <xacro:property name="box_mass" value="0.1"/> <!-- box mass -->
-    <xacro:property name="W_x" value="0.066"/> <!-- wheel axis x-offset from centre -->
-    <xacro:property name="W_z" value="0.022"/> <!-- wheel axis z-offset from bottom -->
-    <xacro:property name="W_y" value="0.122"/> <!-- wheel half separation -->
-    <xacro:property name="W_D" value="0.065"/> <!-- wheel diameter -->
-    <xacro:property name="W_h" value="0.026"/> <!-- wheel width -->
-    <xacro:property name="W_mass" value="0.1"/> <!-- wheel mass -->
-    <xacro:property name="c_x" value="0.024"/> <!-- caster centre x-offset from edge -->
-    <xacro:property name="c_y" value="0.024"/> <!-- caster centre y-offset from edge -->
-    <xacro:property name="c_z" value="0.052"/> <!-- caster contact z-offset from bottom -->
-    <xacro:property name="c_D" value="0.016"/> <!-- caster diameter -->
-    <xacro:property name="c_mass" value="0.1"/> <!-- caster mass -->
-    <xacro:property name="m_y" value="0.04"/> <!-- motor y-offset from centre-->
-    <xacro:property name="m_h" value="0.06"/> <!-- motor length -->
-    <xacro:property name="m_D" value="0.02"/> <!-- motor body diameter -->
-    <xacro:property name="m_l" value="0.009"/> <!-- motor coupling length -->
-    <xacro:property name="m_d" value="0.011"/> <!-- motor coupling diameter -->
-    <xacro:property name="m_mass" value="0.1"/> <!-- motor mass -->
     <!-- BASE LINK -->
     <link name="base_link">
@@ -43,5 +21,5 @@
             </geometry>
             <origin xyz="${L_x/2} 0 ${L_z/2}" />
-            <material name="light_gray" />
+            <material name="green" />
         </visual>
         <collision>
@@ -55,4 +33,7 @@
         </xacro:inertial_box>
     </link>
+    <gazebo reference="chassis_link">
+        <material>Gazebo/Green</material>
+    </gazebo>
     <!-- LEFT WHEEL LINK -->
     <joint name="left_wheel_joint" type = "continuous">
@@ -78,4 +59,7 @@
         </xacro:inertial_cylinder>
     </link>
+    <gazebo reference="left_wheel_link">
+        <material>Gazebo/Blue</material>
+    </gazebo>
     <!-- RIGHT WHEEL LINK -->
     <joint name="right_wheel_joint" type = "continuous">
@@ -101,4 +85,7 @@
         </xacro:inertial_cylinder>
     </link>
+    <gazebo reference="right_wheel_link">
+        <material>Gazebo/Blue</material>
+    </gazebo>
 <!-- LEFT CASTER WHEEL LINK -->
     <joint name="left_caster_wheel_joint" type = "fixed">
@@ -112,5 +99,5 @@
                 <sphere radius="${c_D/2}" />
             </geometry>
-            <material name="light_gray" />
+            <material name="yellow" />
         </visual>
         <collision>
@@ -123,4 +110,9 @@
         </xacro:inertial_sphere>
     </link>
+    <gazebo reference="left_caster_wheel_link">
+        <material>Gazebo/Yellow</material>
+        <mu1 value="0.0001" />
+        <mu2 value="0.0001" />
+    </gazebo>
 <!-- RIGHT CASTER WHEEL LINK -->
     <joint name="right_caster_wheel_joint" type = "fixed">
@@ -134,5 +126,5 @@
                 <sphere radius="${c_D/2}" />
             </geometry>
-            <material name="light_gray" />
+            <material name="yellow" />
         </visual>
         <collision>
@@ -145,4 +137,9 @@
         </xacro:inertial_sphere>
     </link>
+    <gazebo reference="right_caster_wheel_link">
+        <material>Gazebo/Yellow</material>
+        <mu1 value="0.0001" />
+        <mu2 value="0.0001" />
+    </gazebo>
     <!-- LEFT MOTOR LINK -->
     <joint name="left_motor_joint" type = "fixed">
@@ -157,5 +154,5 @@
             </geometry>
             <origin xyz="0 0 0" />
-            <material name="light_gray" />
+            <material name="red" />
         </visual>
         <visual>
@@ -164,5 +161,5 @@
             </geometry>
             <origin xyz="0 0 ${(m_h+m_l)/2}" />
-            <material name="yellow" />
+            <material name="red" />
         </visual>
         <collision>
@@ -175,4 +172,7 @@
         </xacro:inertial_cylinder>
     </link>
+    <gazebo reference="left_motor_link">
+        <material>Gazebo/Red</material>
+    </gazebo>
     <!-- RIGHT MOTOR LINK -->
     <joint name="right_motor_joint" type = "fixed">
@@ -187,5 +187,5 @@
             </geometry>
             <origin xyz="0 0 0" />
-            <material name="light_gray" />
+            <material name="red" />
         </visual>
         <visual>
@@ -194,5 +194,5 @@
             </geometry>
             <origin xyz="0 0 ${(m_h+m_l)/2}" />
-            <material name="yellow" />
+            <material name="red" />
         </visual>
         <collision>
@@ -205,3 +205,6 @@
         </xacro:inertial_cylinder>
     </link>
+    <gazebo reference="right_motor_link">
+        <material>Gazebo/Red</material>
+    </gazebo>
 </robot>
