Commit message: Adjust masses to improve behaviour - values are not real though

File: manolobot_uno/description/properties.xacro (robot description, xacro)
@@ -5,5 +5,5 @@
     <xacro:property name="L_y" value="0.19"/> <!-- box width -->
     <xacro:property name="L_z" value="0.124"/> <!-- box height -->
-    <xacro:property name="box_mass" value="0.1"/> <!-- box mass -->
+    <xacro:property name="box_mass" value="0.05"/> <!-- box mass -->
     <!-- wheels -->
     <xacro:property name="W_x" value="0.066"/> <!-- wheel axis x-offset from centre -->
@@ -12,5 +12,5 @@
     <xacro:property name="W_D" value="0.065"/> <!-- wheel diameter -->
     <xacro:property name="W_h" value="0.026"/> <!-- wheel width -->
-    <xacro:property name="W_mass" value="0.1"/> <!-- wheel mass -->
+    <xacro:property name="W_mass" value="0.05"/> <!-- wheel mass -->
     <!-- casters -->
     <xacro:property name="c_x" value="0.024"/> <!-- caster centre x-offset from edge -->
@@ -18,5 +18,5 @@
     <xacro:property name="c_z" value="0.052"/> <!-- caster contact z-offset from bottom -->
     <xacro:property name="c_D" value="0.016"/> <!-- caster diameter -->
-    <xacro:property name="c_mass" value="0.1"/> <!-- caster mass -->
+    <xacro:property name="c_mass" value="0.05"/> <!-- caster mass -->
     <!-- motors -->
     <xacro:property name="m_y" value="0.04"/> <!-- motor y-offset from centre-->
@@ -25,4 +25,4 @@
     <xacro:property name="m_l" value="0.009"/> <!-- motor coupling length -->
     <xacro:property name="m_d" value="0.011"/> <!-- motor coupling diameter -->
-    <xacro:property name="m_mass" value="0.1"/> <!-- motor mass -->
+    <xacro:property name="m_mass" value="0.05"/> <!-- motor mass -->
 </robot>

Commit message: Add Lidar to robot model
* description/lidar.xacro: new file to define Lidar properties
* description/properties.xacro: rename box dimensions from L_x L_y L_z
  to box_x box_y box_z and leave L_ prefix for lidar
* description/robot_core.xacro and robot.urdf.xacro: modify accordingly
* worlds/cones.world: a sample world with cones

File: manolobot_uno/description/properties.xacro (robot description, xacro)
@@ -2,7 +2,7 @@
 <robot xmlns:xacro="http://www.ros.org/wiki/xacro" >
     <!-- box -->
-    <xacro:property name="L_x" value="0.29"/> <!-- box length -->
-    <xacro:property name="L_y" value="0.19"/> <!-- box width -->
-    <xacro:property name="L_z" value="0.124"/> <!-- box height -->
+    <xacro:property name="box_x" value="0.29"/> <!-- box length -->
+    <xacro:property name="box_y" value="0.19"/> <!-- box width -->
+    <xacro:property name="box_z" value="0.124"/> <!-- box height -->
     <xacro:property name="box_mass" value="0.05"/> <!-- box mass -->
     <!-- wheels -->
@@ -16,5 +16,5 @@
     <xacro:property name="c_x" value="0.024"/> <!-- caster centre x-offset from edge -->
     <xacro:property name="c_y" value="0.024"/> <!-- caster centre y-offset from edge -->
-    <xacro:property name="c_z" value="0.052"/> <!-- caster contact z-offset from bottom -->
+    <xacro:property name="c_z" value="0.049"/> <!-- caster contact z-offset from bottom -->
     <xacro:property name="c_D" value="0.016"/> <!-- caster diameter -->
     <xacro:property name="c_mass" value="0.05"/> <!-- caster mass -->
@@ -26,3 +26,9 @@
     <xacro:property name="m_d" value="0.011"/> <!-- motor coupling diameter -->
     <xacro:property name="m_mass" value="0.05"/> <!-- motor mass -->
+    <!--lidar -->
+    <xacro:property name="L_x" value="0.0"/> <!-- Lidar x-offset from box centre -->
+    <xacro:property name="L_z" value="0.023"/> <!-- Lidar z-offset from box top -->
+    <xacro:property name="L_D" value="0.038"/> <!-- Lidar head diameter -->
+    <xacro:property name="L_h" value="0.013"/> <!-- Lidar unit height -->
+    <xacro:property name="L_mass" value="0.0042"/> <!-- Lidar mass -->
 </robot>

File: manolobot_uno/description/robot.urdf.xacro (robot description, xacro)
@@ -7,3 +7,5 @@
     <!-- GAZEBO -->
     <xacro:include filename="gazebo_control.xacro" />
+    <!-- LIDAR -->
+    <xacro:include filename="lidar.xacro" />
 </robot>

File: manolobot_uno/description/robot_core.xacro (robot description, xacro)
@@ -13,26 +13,26 @@
         <parent link="base_link" />
         <child link="chassis_link" />
-        <origin xyz="${W_x-L_x/2} 0 ${W_z}" />
+        <origin xyz="${W_x-box_x/2} 0 ${W_z}" />
     </joint>
     <link name="chassis_link">
         <visual>
             <geometry>
-                <box size="${L_x} ${L_y} ${L_z}"/>
-            </geometry>
-            <origin xyz="${L_x/2} 0 ${L_z/2}" />
-            <material name="green" />
-        </visual>
-        <collision>
-            <geometry>
-                <box size="${L_x} ${L_y} ${L_z}"/>
-            </geometry>
-            <origin xyz="${L_x/2} 0 ${L_z/2}" />
-        </collision>
-        <xacro:inertial_box mass="${box_mass}" x="${L_x}" y="${L_y}" z="${L_z}">
-            <origin xyz="${L_x/2} 0 ${L_z/2}" rpy="0 0 0" />
+                <box size="${box_x} ${box_y} ${box_z}"/>
+            </geometry>
+            <origin xyz="${box_x/2} 0 ${box_z/2}" />
+            <material name="white" />
+        </visual>
+        <collision>
+            <geometry>
+                <box size="${box_x} ${box_y} ${box_z}"/>
+            </geometry>
+            <origin xyz="${box_x/2} 0 ${box_z/2}" />
+        </collision>
+        <xacro:inertial_box mass="${box_mass}" x="${box_x}" y="${box_y}" z="${box_z}">
+            <origin xyz="${box_x/2} 0 ${box_z/2}" rpy="0 0 0" />
         </xacro:inertial_box>
     </link>
     <gazebo reference="chassis_link">
-        <material>Gazebo/Green</material>
+        <material>Gazebo/White</material>
     </gazebo>
     <!-- LEFT WHEEL LINK -->
@@ -48,5 +48,5 @@
                 <cylinder radius="${W_D/2}" length="${W_h}" />
             </geometry>
-            <material name="dark_gray" />
+            <material name="blue" />
         </visual>
         <collision>
@@ -74,5 +74,5 @@
                 <cylinder radius="${W_D/2}" length="${W_h}" />
             </geometry>
-            <material name="dark_gray" />
+            <material name="blue" />
         </visual>
         <collision>
@@ -92,5 +92,5 @@
         <parent link="chassis_link" />
         <child link="left_caster_wheel_link" />
-        <origin xyz="${L_x-c_x} ${L_y/2-c_y} -${c_z}" />
+        <origin xyz="${box_x-c_x} ${box_y/2-c_y} ${-c_z}" />
     </joint>
     <link name="left_caster_wheel_link">
@@ -99,5 +99,5 @@
                 <sphere radius="${c_D/2}" />
             </geometry>
-            <material name="yellow" />
+            <material name="orange" />
         </visual>
         <collision>
@@ -111,13 +111,13 @@
     </link>
     <gazebo reference="left_caster_wheel_link">
-        <material>Gazebo/Yellow</material>
+        <material>Gazebo/Orange</material>
         <mu1 value="0.0001" />
         <mu2 value="0.0001" />
     </gazebo>
-<!-- RIGHT CASTER WHEEL LINK -->
+<!-- RIGHT CASTER WHEEL LINK     -->
     <joint name="right_caster_wheel_joint" type = "fixed">
         <parent link="chassis_link" />
         <child link="right_caster_wheel_link" />
-        <origin xyz="${L_x-c_x} ${-L_y/2+c_y} -${c_z}" />
+        <origin xyz="${box_x-c_x} ${-box_y/2+c_y} ${-c_z}" />
     </joint>
     <link name="right_caster_wheel_link">

Commit message: Add camera to robot model
    * description/camera.xacro: new file to define camera properties
    * description/properties.xacro: add camera properties with cam_
      prefix
    * description/robot.urdf.xacro: include camera.xacro
    * description/robot_core.xacro: change color of caster wheel
    * BOM/pi_camera.md: Add notes on cameras in ROS
    * config/bot_with_sensors.rviz: RVIZ config file for robot with
      sensors
    * worlds/cones.world: recreated to fix issue

    This setup was used to record the video gazebo2.mp4. The robot
    - operated with the gamepad - drives around a field of cones and
    shows output of camera and lidar.

File: manolobot_uno/description/properties.xacro (robot description, xacro)
@@ -32,3 +32,10 @@
     <xacro:property name="L_h" value="0.013"/> <!-- Lidar unit height -->
     <xacro:property name="L_mass" value="0.0042"/> <!-- Lidar mass -->
+    <!--camera -->
+    <xacro:property name="cam_x" value="0.0"/> <!-- Camera x-offset from box front face -->
+    <xacro:property name="cam_z" value="-0.03"/> <!-- Lidar z-offset from box top -->
+    <xacro:property name="cam_dx" value="0.01"/> <!-- Camera box thickness -->
+    <xacro:property name="cam_dy" value="0.04"/> <!-- Camera box width -->
+    <xacro:property name="cam_dz" value="0.03"/> <!-- Camera box height -->
+    <xacro:property name="cam_mass" value="0.002"/> <!-- Camera mass -->
 </robot>

File: manolobot_uno/description/robot.urdf.xacro (robot description, xacro)
@@ -9,3 +9,5 @@
     <!-- LIDAR -->
     <xacro:include filename="lidar.xacro" />
+    <!-- CAMERA -->
+    <xacro:include filename="camera.xacro" />
 </robot>

File: manolobot_uno/description/robot_core.xacro (robot description, xacro)
@@ -99,5 +99,5 @@
                 <sphere radius="${c_D/2}" />
             </geometry>
-            <material name="orange" />
+            <material name="yellow" />
         </visual>
         <collision>
@@ -111,5 +111,5 @@
     </link>
     <gazebo reference="left_caster_wheel_link">
-        <material>Gazebo/Orange</material>
+        <material>Gazebo/Yellow</material>
         <mu1 value="0.0001" />
         <mu2 value="0.0001" />
