Commit message: Spheres as collision for wheels to reduce drift in gazebo

File: manolobot_uno/description/robot_core.xacro (robot description, xacro)
@@ -52,5 +52,5 @@
         <collision>
             <geometry>
-                <cylinder radius="${W_D/2}" length="${W_h}" />
+                <sphere radius="${W_D/2}" />
             </geometry>
         </collision>
@@ -78,5 +78,5 @@
         <collision>
             <geometry>
-                <cylinder radius="${W_D/2}" length="${W_h}" />
+                <sphere radius="${W_D/2}" />
             </geometry>
         </collision>
